Commit message: Harden photo-matched B2-W Z1 asset

File: source/LeggedManip_Lab/LeggedManip_Lab/assets/b2w_z1/source/b2w_z1.urdf (robot description, URDF)
Before this commit: robot b2w_z1, 35 links, 34 joints
Links:
- added link tcp_frame; visual sphere radius=0.000001
Joints:
- added joint tcp_fixed_joint: type fixed, parent gripper_stator, child tcp_frame, origin xyz=0.145000 0.000000 0.000000 rpy=0.000000 0.000000 0.000000
- joint z1_mount_joint: origin xyz=0.211000 0.000000 0.110000 rpy=0 0 0 -> xyz=0.211000 0.000000 0.110000 rpy=0.000000 0.000000 0.000000
