Commit message: feat: complete staged B2W Z1 door opening baseline

File: source/LeggedManip_Lab/LeggedManip_Lab/assets/door/door_with_lever.urdf (robot description, URDF)
Before this commit: robot door_with_lever, 4 links, 3 joints
Links:
- link door_panel: geometry collision box size=0.050 0.90 1.98; visual box size=0.050 0.90 1.98
- link handle_grasp: mass None -> 0.001
Joints:
- joint door_hinge: limit lower=0.0 upper=1.65 effort=180 velocity=1.5 -> lower=-0.05 upper=1.65 effort=180 velocity=1.5
